File: hardware/KiCAD/PCB_Aquarium_v2/Food.kicad_sch (KiCad schematic)
At the start: 5 parts, among them J10 Conn_01x03, J14 Conn_01x03, J15 Conn_01x03, J16 Conn_01x03, J17 Conn_01x03

Commit message: PCB principal finis
Parts:
- removed J17: Conn_01x03, symbol Connector_Generic:Conn_01x03
- added C807, C808, C809: 1u, Capacitor_SMD:C_0603_1608Metric, symbol Device:C_Small
- added C810: D8L6.5_865090349007, Capacitor_SMD_Wurth:CP_Wurth_WCAP-ASLU-D8L6.5, symbol Capacitor_Wurth_WCAP-ASLU:D8L6.5_865090349007
- added C811: 100n, Capacitor_SMD:C_0402_1005Metric, symbol Device:C_Small
- J801: renamed from J14; footprint (none) -> Connector_JST:JST_SH_BM03B-SRSS-TB_1x03-1MP_P1.00mm_Vertical; symbol Connector_Generic:Conn_01x03 -> my_lib:JST_SH_3_Vertical
- J802: renamed from J15; footprint (none) -> Connector_JST:JST_SH_BM03B-SRSS-TB_1x03-1MP_P1.00mm_Vertical; symbol Connector_Generic:Conn_01x03 -> my_lib:JST_SH_3_Vertical
- J803: renamed from J16; footprint (none) -> Connector_JST:JST_SH_BM03B-SRSS-TB_1x03-1MP_P1.00mm_Vertical; symbol Connector_Generic:Conn_01x03 -> my_lib:JST_SH_3_Vertical
- J805: renamed from J10; footprint (none) -> Connector_JST:JST_PH_B3B-PH-K_1x03_P2.00mm_Vertical
Connections:
- net +3.3V: now also C807.1, C808.1, C809.1
- net +5V: now also C810.1, C811.1
- net GND: now also J801.MP (GND), J802.MP (GND), J803.MP (GND), C807.2, C808.2, C809.2, C810.2, C811.2
