File: hardware/KiCAD/PCB_Aquarium_v2/Pump.kicad_sch (KiCad schematic)
At the start: 12 parts, among them J22 Conn_01x02, J23 Conn_01x02, Q1 NMOS, Q2 NMOS

Commit message: PCB principal finis
Parts:
- removed C28, C29: 1u, Capacitor_SMD:C_0603_1608Metric, symbol Device:C
- removed J22, J23: Conn_01x02, Connector_JST:JST_EH_B2B-EH-A_1x02_P2.50mm_Vertical, symbol Connector_Generic:Conn_01x02
- added D701, D702, D703, D704: D_Schottky, mylib:FSV330AF, symbol Device:D_Schottky
- added J703, J704: Conn_01x02, Connector_JST:JST_SH_BM02B-SRSS-TB_1x02-1MP_P1.00mm_Vertical, symbol my_lib:JST_SH_2_Vertical
- added Q703, Q704: NMOS, Package_TO_SOT_SMD:SOT-23, symbol Simulation_SPICE:NMOS
- added R705, R707: 1k, Resistor_SMD:R_0402_1005Metric, symbol Device:R
- added R706, R708: 10k, Resistor_SMD:R_0402_1005Metric, symbol Device:R
- J701: renamed from J22; footprint Connector_JST:JST_EH_B2B-EH-A_1x02_P2.50mm_Vertical -> Connector_JST:JST_SH_BM02B-SRSS-TB_1x02-1MP_P1.00mm_Vertical; symbol Connector_Generic:Conn_01x02 -> my_lib:JST_SH_2_Vertical
- J702: renamed from J23; footprint Connector_JST:JST_EH_B2B-EH-A_1x02_P2.50mm_Vertical -> Connector_JST:JST_SH_BM02B-SRSS-TB_1x02-1MP_P1.00mm_Vertical; symbol Connector_Generic:Conn_01x02 -> my_lib:JST_SH_2_Vertical
- Q701: renamed from Q1; MPN SQ2310ES -> SQ2310ES-T1_BE3
- Q702: renamed from Q2; MPN SQ2310ES -> SQ2310ES-T1_BE3
- renumbered R1 to R701, R2 to R702, R3 to R703, R4 to R704
Connections:
- net +12V: now also D701.1 (K), D702.1 (K), D703.1 (K), D704.1 (K), J703.1, J704.1
- net GND: now also J701.MP (GND), J702.MP (GND), J703.MP (GND), J704.MP (GND), Q703.3 (S), Q704.3 (S), R706.2, R708.2
- net at J701.2, Q701.1 (D): now also D701.2 (A)
- net at J702.2, Q702.1 (D): now also D702.2 (A)
- new net: D704.2 (A), J704.2, Q704.1 (D)
- new net: D703.2 (A), J703.2, Q703.1 (D)
- new net: Q704.2 (G), R707.1, R708.1
- new net: Q703.2 (G), R705.1, R706.1
- new net GPIO_Pump_3: R705.2
- new net GPIO_Pump_4: R707.2
