File: hardware/KiCAD/PCB_Aquarium_v2/Voltage.kicad_sch (KiCad schematic)
At the start: 10 parts, among them U2 173010578, U3 AZ1117-3.3

Commit message: PCB principal finis
Parts:
- added C303: 470u, Capacitor_SMD:C_Elec_10x10.2, symbol Device:C_Small
- renumbered C38 to C301, C39 to C302, D1 to D301, D2 to D302, D3 to D303, R5 to R301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
Connections:
- net +12V: now also C303.1
- net GND: now also C303.2
