File: hardware/KiCAD/PCB_Aquarium_v2/PCB_Aquarium_v2.kicad_sch (KiCad schematic)
At the start: 0 parts

Commit message: update sch pcb
Parts:
- added C11: 1u, Capacitor_SMD:C_0603_1608Metric, symbol Device:C
- added C20: 4u7, Capacitor_SMD:C_0603_1608Metric, symbol Device:C_Small
- added C21, C24, C25, C27, C4, C6: 100n, Capacitor_SMD:C_0402_1005Metric, symbol Device:C_Small
- added C22, C30: 1u, Capacitor_SMD:C_0402_1005Metric, symbol Device:C_Small
- added C5: 10u, Capacitor_SMD:C_0603_1608Metric, symbol Device:C_Small
- added C7: 10n, Capacitor_SMD:C_0402_1005Metric, symbol Device:C_Small
- added C8: 220n, symbol Device:C_Small
- added C9: 100n, symbol Device:C_Small
- added D20: ~, Diode_SMD:D_SOD-523, symbol my_lib:VESD05A1-02V-G3-08
- added F1: 1A, Fuse:Fuse_2920_7451Metric, symbol Device:Polyfuse_Small
- added H1, H2, H3, H4: MountingHole_Pad, MountingHole:MountingHole_3.2mm_M3_Pad_Via, symbol Mechanical:MountingHole_Pad
- added J1, J21: Conn_01x02, symbol Connector_Generic:Conn_01x02
- added J103, J18, J19, J20: Conn_01x03, Connector_JST:JST_EH_B3B-EH-A_1x03_P2.50mm_Vertical, symbol Connector_Generic:Conn_01x03
- added J11, J12, J13: Conn_01x03, symbol Connector_Generic:Conn_01x03
- added J24: Conn_01x04, Connector_THT_Wurth:J_Wurth_WR-WTB_62000411722, symbol Connector_Generic:Conn_01x04
- added J35: Conn_ST_STDC14, Connector_PinHeader_1.27mm:PinHeader_2x07_P1.27mm_Vertical_SMD, symbol Connector:Conn_ST_STDC14
- added L1: 39n, Inductor_SMD:L_0603_1608Metric, symbol Device:L_Small
- added R8: 25k, symbol Device:R_Small
- added SW1: SW_SPDT, symbol Switch:SW_SPDT
- added U1: ~, symbol my_lib:A4988
- added U5: STM32G474RETx, Package_QFP:LQFP-64_10x10mm_P0.5mm, symbol MCU_ST_STM32G4:STM32G474RETx
Connections:
- new net: C9.1, U1.4 (CP1)
- new net: C9.2, U1.5 (CP2)
- new net: R8.2, U1.13 (ROSC)
- new net: C8.1, U1.8 (VREG)
- new net: J1.2 (Pin_2), SW1.2 (B)
- new net +12V: J103.2 (Pin_2), J18.2 (Pin_2), J19.2 (Pin_2), J21.1 (Pin_1), SW1.1 (A)
- new net +3.3V: C20.1, C21.1, C22.1, C24.1, C25.1, C27.1, C6.1, J11.2 (Pin_2), J12.2 (Pin_2), J13.2 (Pin_2), J35.3 (VCC), L1.1, U5.1 (VBAT), U5.16 (VDD), U5.28 (VREF+), U5.32 (VDD), U5.48 (VDD), U5.64 (VDD)
- new net +3.3VA: C30.2, C7.1, L1.2, U5.29 (VDDA)
- new net +5V: C11.1, F1.2, J20.2 (Pin_2)
- new net 5V_Rpi: C4.1, C5.1, D20.2 (A2), F1.1, J24.2 (Pin_2)
- new net GND: C11.2, C20.2, C21.2, C22.2, C24.2, C25.2, C27.2, C30.1, C4.2, C5.2, C6.2, C7.2, C8.2, D20.1 (A1), H1.1, H2.1, H3.1, H4.1, J1.1 (Pin_1), J103.1 (Pin_1), J11.3 (Pin_3), J12.3 (Pin_3), J13.3 (Pin_3), J18.1 (Pin_1), J19.1 (Pin_1), J20.1 (Pin_1), J21.2 (Pin_2), J24.1 (Pin_1), J35.11 (GNDDetect), J35.5 (GND), J35.7 (GND), U1.0 (PAD), U1.18 (GND), U1.3 (GND), U5.15 (VSS), U5.27 (VSSA), U5.31 (VSS), U5.47 (VSS), U5.63 (VSS)
- new net NRST: J35.12 (~{RST})
- new net Output: J20.3 (Pin_3)
- new net SWCLK: J35.6 (JCLK/SWCLK)
- new net SWDIO: J35.4 (JTMS/SWDIO)
- new net UART_DEBUG_RX: J35.13 (VCP_RX)
- new net UART_DEBUG_TX: J35.14 (VCP_TX)
- new net UART_HD_XL430: J103.3 (Pin_3), J18.3 (Pin_3), J19.3 (Pin_3)
- new net UART_Pi_Zero_RX: J24.3 (Pin_3)
- new net UART_Pi_Zero_TX: J24.4 (Pin_4)
- new net hatchway_PWM_1: J11.1 (Pin_1)
- new net hatchway_PWM_2: J12.1 (Pin_1)
- new net hatchway_PWM_3: J13.1 (Pin_1)
- no-connect marks 0 -> 4
Other:
- added sheet Fan (Fan.kicad_sch)
- added sheet Food (Food.kicad_sch)
- added sheet Neopixel (Neopixel.kicad_sch)
- added sheet Pump (Pump.kicad_sch)
- added sheet Screen (Screen.kicad_sch)
- added sheet Voltage (Voltage.kicad_sch)
- added sheet Water_level_sensor (water.kicad_sch)
- note added: "MOUNTING HOLES"
- note added: "Pi Zero 2W"
- note added: "t_off = R_osc/825 in us"

Commit message: PCB principal finis
Parts:
- removed C8: 220n, symbol Device:C_Small
- removed C9: 100n, symbol Device:C_Small
- removed J103, J18, J19: Conn_01x03, Connector_JST:JST_EH_B3B-EH-A_1x03_P2.50mm_Vertical, symbol Connector_Generic:Conn_01x03
- removed J11, J12, J13: Conn_01x03, symbol Connector_Generic:Conn_01x03
- removed J21: Conn_01x02, symbol Connector_Generic:Conn_01x02
- removed R8: 25k, symbol Device:R_Small
- removed U1: ~, symbol my_lib:A4988
- added C102: D8L6.5_865090349007, Capacitor_SMD_Wurth:CP_Wurth_WCAP-ASLU-D8L6.5, symbol Capacitor_Wurth_WCAP-ASLU:D8L6.5_865090349007
- added C103, C107: 100n, Capacitor_SMD:C_0402_1005Metric, symbol Device:C_Small
- added J102: Conn_01x03, Connector_JST:JST_PH_B3B-PH-K_1x03_P2.00mm_Vertical, symbol Connector_Generic:Conn_01x03
- added R101, R102: 4k7, Resistor_SMD:R_0201_0603Metric, symbol Device:R_Small
- added SW101: ~, mylib:WS-TASV SMT Tact Switch 3.0 x 2.6 mm, symbol my_lib:WS-TASV_SMT_Tact_Switch_3.0_x_2.6_mm
- D101: renamed from D20; MPW (none) -> VESD05A1-02V-G3-08
- J101: renamed from J20; footprint Connector_JST:JST_EH_B3B-EH-A_1x03_P2.50mm_Vertical -> Connector_JST:JST_SH_BM03B-SRSS-TB_1x03-1MP_P1.00mm_Vertical; symbol Connector_Generic:Conn_01x03 -> my_lib:JST_SH_3_Vertical
- J103: renamed from J1; footprint (none) -> Connector_AMASS:AMASS_XT30U-M_1x02_P5.0mm_Vertical
- J104: renamed from J24; footprint Connector_THT_Wurth:J_Wurth_WR-WTB_62000411722 -> Connector_JST:JST_PH_B4B-PH-K_1x04_P2.00mm_Vertical
- SW102: renamed from SW1; footprint (none) -> mylib:SW_Wurth_WS-TOTV_472123020421
- renumbered C11 to C101, C20 to C104, C21 to C105, C22 to C106, C24 to C108, C25 to C109, C27 to C110, C6 to C111, C7 to C112, C30 to C113, C4 to C114, C5 to C115, F1 to F101, H1 to H101, H2 to H102, H3 to H103, H4 to H104, J35 to J105, L1 to L101, U5 to U101
Connections:
- net +5V: now also C102.1, C103.1, J102.1 (Pin_1), R101.1, R102.1
- net GND: now also J101.MP (GND), U101.61 (PB8), C102.2, C103.2, C107.2, J102.3 (Pin_3), SW101.3, SW101.4, SW101.5, SW101.6 (GND)
- net NRST: now also U101.7 (PG10), C107.1, SW101.1, SW101.2
- net Output: now also U101.26 (PB2)
- net SWCLK: now also U101.50 (PA14)
- net SWDIO: now also U101.49 (PA13)
- net UART_DEBUG_RX: now also U101.17 (PA3)
- net UART_DEBUG_TX: now also U101.14 (PA2)
- net UART_Pi_Zero_RX: now also U101.33 (PB11)
- net UART_Pi_Zero_TX: now also U101.30 (PB10)
- net hatchway_PWM_1: now also U101.51 (PA15)
- net hatchway_PWM_2: now also U101.38 (PC6)
- net hatchway_PWM_3: now also U101.40 (PC8)
- net food_PWM_3: now reaches U101.10 (PC2)
- net food_PWM_2: now reaches U101.11 (PC3)
- net food_PWM_1: now reaches U101.12 (PA0)
- net heater_STEP: now reaches U101.18 (PA4)
- net heater_SLEEP: now reaches U101.19 (PA5)
- net GPIO_Pump_4: now reaches U101.2 (PC13)
- net heater_RESET: now reaches U101.20 (PA6)
- net GPIO_Pump_3: now reaches U101.3 (PC14)
- net Water_int_1: now reaches U101.34 (PB12)
- net Water_int_2: now reaches U101.35 (PB13)
- net Water_int_3: now reaches U101.36 (PB14)
- net GEAR_PWM_4: now reaches U101.37 (PB15)
- net GEAR_PWM_2: now reaches U101.39 (PC7)
- net GEAR_PWM_5: now reaches U101.41 (PC9)
- net Screen_SDA: now reaches U101.42 (PA8)
- net Screen_SDA: now also R101.2
- net Screen_SCL: now reaches U101.43 (PA9)
- net Screen_SCL: now also R102.2
- net Screen_RESET: now reaches U101.44 (PA10)
- net GPIO_Pump_1: now reaches U101.45 (PA11)
- net GPIO_Pump_2: now reaches U101.46 (PA12)
- net heater_EN: now reaches U101.5 (PF0)
- net GEAR_PWM_1: now reaches U101.52 (PC10)
- net Reverse_PWM_1: now reaches U101.57 (PB4)
- net GEAR_PWM_3: now reaches U101.58 (PB5)
- net Reverse_PWM_3: now reaches U101.59 (PB6)
- net heater_DIR: now reaches U101.6 (PF1)
- net GEAR_PWM_6: now reaches U101.60 (PB7)
- net Reverse_PWM_2: now reaches U101.62 (PB9)
- net LED_externe_PWM: now reaches U101.8 (PC0)
- net LED_interne_PWM: now reaches U101.9 (PC1)
- net LED_interne_PWM: now also J102.2 (Pin_2)
- no-connect marks 4 -> 15
Other:
- removed sheet Neopixel
- added sheet Drop_Test (Drop_Test.kicad_sch)
- added sheet heater (heater.kicad_sch)
- sheet Food ports: added LED_externe_PWM, food_PWM_1, food_PWM_2, food_PWM_3; removed none
- sheet Pump ports: added GPIO_Pump_1, GPIO_Pump_2, GPIO_Pump_3, GPIO_Pump_4; removed none
- sheet Screen ports: added Screen_RESET, Screen_SCL, Screen_SDA; removed none
- note added: "Sonde PH"
- note removed: "t_off = R_osc/825 in us"
- moved on the sheet: C101

Commit message: PCB Neopixel
Parts:
- added TP101, TP102: TestPoint, TestPoint:TestPoint_Pad_D2.0mm, symbol Connector:TestPoint
Connections:
- net Screen_SCL: now also TP101.1
- net Screen_SDA: now also TP102.1
Changed lines of the file:
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@@
 	)
 	(junction
+		(at 191.77 68.58)
+		(diameter 0)
+		(color 0 0 0 0)
+	)
+	(junction
 		(at 267.97 26.67)
 		(diameter 0)
@@
 	)
 	(junction
+		(at 195.58 71.12)
+		(diameter 0)
+		(color 0 0 0 0)
+	)
+	(junction
 		(at 259.08 147.32)
 		(diameter 0)
@@
 	(wire
 		(pts
-			(xy 194.31 68.58) (xy 167.64 68.58)
+			(xy 194.31 68.58) (xy 191.77 68.58)
 		)
 		(stroke
@@
 	(wire
 		(pts
+			(xy 195.58 71.12) (xy 167.64 71.12)
+		)
+		(stroke
+			(width 0)
+			(type default)
+		)
+	)
+	(wire
+		(pts
 			(xy 260.35 21.59) (xy 267.97 21.59)
 		)
@@
 	(wire
 		(pts
+			(xy 191.77 68.58) (xy 167.64 68.58)
+		)
+		(stroke
+			(width 0)
+			(type default)
+		)
+	)
+	(wire
+		(pts
 			(xy 101.6 53.34) (xy 104.14 53.34)
 		)
@@
 	(wire
 		(pts
-			(xy 196.85 71.12) (xy 167.64 71.12)
+			(xy 196.85 71.12) (xy 195.58 71.12)
 		)
 		(stroke
@@
 	)
 	(symbol
+		(lib_id "Connector:TestPoint")
+		(at 191.77 68.58 0)
+		(mirror y)
+		(unit 1)
+		(exclude_from_sim no)
+		(in_bom yes)
+		(on_board yes)
+		(dnp no)
+		(property "Reference" "TP102"
+			(at 189.23 64.0079 0)
+			(effects
+				(font
+					(size 1.27 1.27)
+				)
+				(justify left)
+			)
+		)
+		(property "Value" "TestPoint"
+			(at 189.23 66.5479 0)
+			(effects
+				(font
+					(size 1.27 1.27)
+				)
+				(justify left)
+			)
+		)
+		(property "Footprint" "TestPoint:TestPoint_Pad_D2.0mm"
+			(at 186.69 68.58 0)
+			(effects
+				(font
+					(size 1.27 1.27)
+				)
+				(hide yes)
+			)
+		)
+		(property "Datasheet" "~"
+			(at 186.69 68.58 0)
+			(effects
+				(font
+					(size 1.27 1.27)
+				)
+				(hide yes)
+			)
+		)
+		(property "Description" "test point"
+			(at 191.77 68.58 0)
+			(effects
+				(font
+					(size 1.27 1.27)
+				)
+				(hide yes)
+			)
+		)
+		(pin "1"
+		)
+		(instances
+			(project ""
+				(path "/2dd88866-dc89-46d7-b019-002e9029eb7f"
+					(reference "TP102")
+					(unit 1)
+				)
+			)
+		)
+	)
+	(symbol
 		(lib_id "power:+5V")
 		(at 76.2 180.34 0)
@@
 					(unit 1)
 				)
+			)
+		)
+	)
+	(symbol
+		(lib_id "Connector:TestPoint")
+		(at 195.58 71.12 180)
+		(unit 1)
+		(exclude_from_sim no)
+		(in_bom yes)
+		(on_board yes)
+		(dnp no)
+		(fields_autoplaced yes)
+		(property "Reference" "TP101"
+			(at 198.12 73.1519 0)
+			(effects
+				(font
+					(size 1.27 1.27)
+				)
+				(justify right)
+			)
+		)
+		(property "Value" "TestPoint"
+			(at 198.12 75.6919 0)
+			(effects
+				(font
+					(size 1.27 1.27)
+				)
+				(justify right)
+			)
+		)
+		(property "Footprint" "TestPoint:TestPoint_Pad_D2.0mm"
+			(at 190.5 71.12 0)
+			(effects
+				(font
+					(size 1.27 1.27)
+				)
+				(hide yes)
+			)
+		)
+		(property "Datasheet" "~"
+			(at 190.5 71.12 0)
+			(effects
+				(font
+					(size 1.27 1.27)
+				)
+				(hide yes)
+			)
+		)
+		(property "Description" "test point"
+			(at 195.58 71.12 0)
+			(effects
+				(font
+					(size 1.27 1.27)
+				)
+				(hide yes)
+			)
+		)
+		(pin "1"
+		)
+		(instances
+			(project ""
+				(path "/2dd88866-dc89-46d7-b019-002e9029eb7f"
+					(reference "TP101")
+					(unit 1)
+				)
