File: hardware/KiCAD/PCB_Neopixel/PCB_Neopixel.kicad_sch (KiCad schematic)
At the start: 4 parts, among them J101 Conn_01x01, J102 Conn_01x01, J103 Conn_01x01

Commit message: PCB 100x10
Parts:
- renumbered C101 to C1201, J101 to J1201, J102 to J1202, J103 to J1203
Connections:
- net DO: no longer J1203.1 (Pin_1)
- net DO8: now also J1203.1 (Pin_1)
Other:
- moved on the sheet: C1201, J1201, J1202, J1203
